File: Sluisbrinkie DIVN/divn/divn.kicad_pcb (KiCad board)
At the start: 2 copper layers, 20 x 100 mm, 60 parts, among them J1 Eurorack Power, J4 CLOCK_IN, J5 CLOCK_OUT, J6 CV IN, Q1 BC847C, Q2 BC847C, Q3 BC847C, Q4 BC847C, U1 40106, U16 TL072CD, U3 4013

Commit message: Finish DIVN layout
Parts:
- added H1: MountingHole, MountingHole:MountingHole_3.2mm_M3, F.Cu at (150.0, 67.5)
- moved R28 32.6 mm to (156.0, 100.5), turned to -90 degrees
- moved R29 31.8 mm to (157.0, 100.5), turned to 90 degrees
- moved RV11 31.8 mm to (157.0, 96.5), turned to 180 degrees
- moved Q1 25.8 mm to (146.5, 127.5)
- moved R37 22.0 mm to (149.5, 140.0), turned to 90 degrees
- moved R38 19.8 mm to (151.0, 140.5)
- moved Q4 18.7 mm to (150.5, 143.0)
- moved R44 17.0 mm to (151.0, 89.0), turned to 90 degrees
- moved R45 16.9 mm to (149.5, 88.5)
- moved C30 15.4 mm to (149.5, 89.5)
- moved D9 10.9 mm to (155.0, 109.0), turned to 0 degrees
- moved C22 10.3 mm to (152.0, 99.5), turned to 0 degrees
- moved R30 9.96 mm to (157.0, 112.0), turned to -90 degrees
- moved D5 9.19 mm to (143.5, 89.5)
- moved D10 8.54 mm to (146.5, 130.5)
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Routing:
- net +12V: track 42.2 -> 162.1 mm, vias 0 -> 7
- net GND: track 62.5 -> 2.00 mm, vias 0 -> 93
- net -12V: track 12.7 -> 52.6 mm, vias 0 -> 3
- net Net-(U16A-+): track 44.0 -> 8.91 mm
- net Net-(Q1-B): track 47.0 -> 18.8 mm
- net Net-(U16B--): track 71.2 -> 48.3 mm, vias 2 -> 3
- net Net-(Q4-C): track 26.4 -> 5.04 mm
- net Net-(Q2-C): track 28.9 -> 12.7 mm
- net Net-(U3B-D): track 39.7 -> 54.1 mm
- net Net-(R44-Pad2): track 14.6 -> 2.85 mm
- net Net-(C26-Pad2): track 9.72 -> 3.70 mm
- net Net-(Q4-B): track 7.89 -> 2.56 mm
- net Net-(Q3-B): track 26.9 -> 21.9 mm
- net Net-(R39-Pad2): track 63.0 -> 58.2 mm
- net Net-(U16A--): track 40.8 -> 36.0 mm
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- added copper zone on B.Cu, net GND
