File: Sluisbrinkie DIVN/divn/divn.kicad_sch (KiCad schematic)
At the start: 60 parts, among them J1 Eurorack Power, J4 CLOCK_IN, J5 CLOCK_OUT, J6 CV IN, Q1 BC847C, Q2 BC847C, Q3 BC847C, Q4 BC847C, U1 40106, U16 TL072CD, U3 4013

Commit message: Finish DIVN layout
Parts:
- added H1: MountingHole, MountingHole:MountingHole_3.2mm_M3, symbol Mechanical:MountingHole
Connections:
- no-connect marks 2 -> 3
Other:
- moved on the sheet: C1, C2
